File: Stasis-Robotic-Arm/Stasis-Robotic-Arm.kicad_pcb (KiCad board)
At the start: 2 copper layers, 83 parts, among them J1 Screw_Terminal_01x04, J2 USB_C_Receptacle_USB2.0_14P, J3 Screw_Terminal_01x04, J4 Screw_Terminal_01x04, J5 Screw_Terminal_01x04, J6 Screw_Terminal_01x04, J8 Screw_Terminal_01x03, SW1 Enable, SW2 Reset, U4 NCP1117-3.3_SOT223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

Commit message: Add files via upload
Parts:
- removed BT1: Battery, Connector_Phoenix_GMSTB:PhoenixContact_GMSTBVA_2,5_2-G-7,62_1x02_P7.62mm_Vertical
- removed C49: 100μF, Capacitor_SMD:C_1206_3216Metric
- removed C50: 100nF, Capacitor_SMD:C_0402_1005Metric
- removed R12, R16, R20, R24, R6: 1K, Resistor_SMD:R_0402_1005Metric
- removed R15, R19, R23, R5, R7: 10K, Resistor_SMD:R_0402_1005Metric
- added C38: 100μF, Capacitor_Tantalum_SMD:CP_EIA-6032-28_Kemet-C, F.Cu at (-66.8, 44.1)
- added C39: 100nF, Capacitor_SMD:C_0402_1005Metric, F.Cu at (-96.8, 36.1)
- added D1: PMEG3010EJ, Diode_SMD:D_SOD-123, F.Cu at (-88.7, 45.4)
- added D2: PMEG3010EJ, Diode_SMD:D_SOD-123, F.Cu at (-88.7, 48.8)
- added J7: Screw_Terminal_01x02, Connector_Phoenix_GMSTB:PhoenixContact_GMSTBVA_2,5_2-G-7,62_1x02_P7.62mm_Vertical, F.Cu at (-57.6, 35.3)
- added R27: 100K, Resistor_SMD:R_0402_1005Metric, F.Cu at (-46.4, 43.1)
- added R28: 100K, Resistor_SMD:R_0402_1005Metric, F.Cu at (-46.4, 45.1)
- added R29: 1K, Resistor_SMD:R_0402_1005Metric, F.Cu at (-46.4, 47.1)
- added R30: 1K, Resistor_SMD:R_0402_1005Metric, F.Cu at (-46.4, 49.1)
- added U10: TVS1400DRV, Package_SON:WSON-6-1EP_2x2mm_P0.65mm_EP1x1.6mm, F.Cu at (-93.5, 49.3)
- added U9: TVS1400DRV, Package_SON:WSON-6-1EP_2x2mm_P0.65mm_EP1x1.6mm, F.Cu at (-93.5, 45.6)
- C13, C18, C23, C4: footprint Capacitor_SMD:C_1206_3216Metric -> Capacitor_Tantalum_SMD:CP_EIA-6032-28_Kemet-C
- C28: value 100μF -> 100uF; footprint Capacitor_SMD:C_1206_3216Metric -> Capacitor_Tantalum_SMD:CP_EIA-6032-28_Kemet-C
- moved J2 134.0 mm to (81.7, 114.9)
- moved R8 40.3 mm to (-49.4, 49.1)
- moved C17 39.6 mm to (-93.4, 35.0)
- moved C22 39.6 mm to (-93.4, 37.5)
- moved C26 39.6 mm to (-99.7, 32.2)
- moved C27 39.6 mm to (-93.4, 40.0)
- moved C29 39.6 mm to (-99.7, 34.2)
- moved C30 39.6 mm to (-99.7, 36.1)
- moved C31 39.6 mm to (-99.7, 38.1)
- moved C32 39.6 mm to (-93.4, 42.5)
- moved C33 39.6 mm to (-99.7, 40.1)
- moved C34 39.6 mm to (-99.7, 42.0)
- moved C35 39.6 mm to (-99.7, 44.0)
- moved C8 39.6 mm to (-93.4, 32.5)
- moved C1 39.6 mm to (-105.4, 32.2)
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Connections:
- net /RXD0 renamed /PDN0-TX
- net /RXD1 renamed /PDN1-TX
- C11 pad 1: +3V3 -> Net-(D1-A)
- C9 pad 1: +3V3 -> Net-(D2-A)
- U1 pad 22: unconnected-(U1-IO14-Pad22) -> /ENN
- U2 pad 2: Net-(U2-ENN) -> /ENN
- U3 pad 2: Net-(U3-ENN) -> /ENN
- U3 pad 25: unconnected-(U3-GND-Pad25) -> GND
- U4 pad 2: +3V3 -> Net-(D2-A)
- U5 pad 2: Net-(U5-ENN) -> /ENN
- U5 pad 25: unconnected-(U5-GND-Pad25) -> GND
- U6 pad 2: Net-(U6-ENN) -> /ENN
- U6 pad 25: unconnected-(U6-GND-Pad25) -> GND
- U7 pad 2: Net-(U7-ENN) -> /ENN
- U7 pad 25: unconnected-(U7-GND-Pad25) -> GND
- U8 pad 2: +3V3 -> Net-(D1-A)
