File: Stasis-Robotic-Arm/Stasis-Robotic-Arm.kicad_sch (KiCad schematic)
At the start: 98 parts, among them J1 Screw_Terminal_01x02, J2 USB_C_Receptacle_USB2.0_14P, J3 Screw_Terminal_01x04, J4 Screw_Terminal_01x04, J5 Screw_Terminal_01x04, J6 Screw_Terminal_01x04, J7 Screw_Terminal_01x04, J8 Screw_Terminal_01x03, SW1 SW_Omron_B3FS, SW2 SW_Omron_B3FS, U4 NCP1117-3.3_SOT223

Commit message: Add files via upload
Parts:
- removed C17, C27, C32, C41, C42, C44, C45, C46: 100nF, Capacitor_SMD:C_0402_1005Metric, symbol Device:C_Small
- removed C21, C30, C39, C48: 2.2μF, Capacitor_SMD:C_0603_1608Metric, symbol Device:C
- removed C22, C40, C43: 100μF, Capacitor_SMD:C_1206_3216Metric, symbol Device:C_Small
- removed C38, C47: 22nF, Capacitor_SMD:C_0402_1005Metric, symbol Device:C_Small
- removed J1: Screw_Terminal_01x02, symbol Connector:Screw_Terminal_01x02
- removed J7: Screw_Terminal_01x04, symbol Connector:Screw_Terminal_01x04
- removed R27: 10K, Resistor_SMD:R_0402_1005Metric, symbol Device:R
- removed R28: 1K, Resistor_SMD:R_0402_1005Metric, symbol Device:R
- removed R29: 100K, Resistor_SMD:R_0402_1005Metric, symbol Device:R
- removed R30, R31: 0.1, Resistor_SMD:R_1206_3216Metric, symbol Device:R
- added BT1: Battery, symbol Device:Battery
- added C17, C22, C27, C32: 2.2μF, Capacitor_SMD:C_0603_1608Metric, symbol Device:C
- added C21: 22nF, symbol Device:C_Small
- added C30: 100nF, Capacitor_SMD:C_0402_1005Metric, symbol Device:C_Small
- added J1: Screw_Terminal_01x04, symbol Connector:Screw_Terminal_01x04
- added U8: NCP1117-3.3_SOT223, Package_TO_SOT_SMD:SOT-223-3_TabPin2, symbol Regulator_Linear:NCP1117-3.3_SOT223
- C10, C6: value 100nF -> 10μF; footprint Capacitor_SMD:C_0402_1005Metric -> (none)
- C11: value 22nF -> 10uF; footprint Capacitor_SMD:C_0402_1005Metric -> (none)
- C13: footprint Capacitor_SMD:C_1206_3216Metric -> (none)
- C14, C19, C24, C33, C35, C36, C37: footprint Capacitor_SMD:C_0402_1005Metric -> (none)
- C16, C31: value 100μF -> 22nF; footprint Capacitor_SMD:C_1206_3216Metric -> (none)
- C18, C23, C28, C4: value 100nF -> 100μF; footprint Capacitor_SMD:C_0402_1005Metric -> (none)
- C20: value 22nF -> 100nF
- C25: value 100μF -> 100nF; footprint Capacitor_SMD:C_1206_3216Metric -> Capacitor_SMD:C_0402_1005Metric
- C26: value 100nF -> 22nF; footprint Capacitor_SMD:C_0402_1005Metric -> (none)
- C29: value 22nF -> 100nF; footprint Capacitor_SMD:C_0402_1005Metric -> (none)
- C3: value 100μF -> 22nF; footprint Capacitor_SMD:C_0402_1005Metric -> (none)
- C34: value 100μF -> 100nF; footprint Capacitor_SMD:C_1206_3216Metric -> (none)
- C5: value 100μF -> 100nF; footprint Capacitor_SMD:C_0402_1005Metric -> (none)
- C9: value 100nF -> 10uF; footprint Capacitor_SMD:C_0402_1005Metric -> (none)
- R12: value 10K -> 1K
- R13, R18: value 1K -> 0.1; footprint Resistor_SMD:R_0402_1005Metric -> Resistor_SMD:R_1206_3216Metric
- R14: value 100K -> 0.1; footprint Resistor_SMD:R_0402_1005Metric -> Resistor_SMD:R_1206_3216Metric
- R15: value 0.1 -> 10K; footprint Resistor_SMD:R_1206_3216Metric -> Resistor_SMD:R_0402_1005Metric
- R16, R20: value 0.1 -> 1K; footprint Resistor_SMD:R_1206_3216Metric -> Resistor_SMD:R_0402_1005Metric
- R17, R22: value 10K -> 0.1; footprint Resistor_SMD:R_0402_1005Metric -> Resistor_SMD:R_1206_3216Metric
- R19, R7: value 100K -> 10K
- R23: value 1K -> 10K
- R24: value 100K -> 1K
- SW1: value SW_Omron_B3FS -> Enable
- SW2: value SW_Omron_B3FS -> Reset
Connections:
- net +3V3: now also C11.1, C15.2, C20.2, C25.2, C9.1, U6.9 (MS1_AD0), C30.2, U8.2 (VO); no longer C19.2, C28.2, C37.2, J2.A4 (VBUS), J2.A9 (VBUS), J2.B4 (VBUS), J2.B9 (VBUS), U5.9 (MS1_AD0)
- net +5V: no longer C10.2, C13.2, C14.2, C15.2, C16.2, C18.2, C23.2, C24.2, C25.2, C26.2, C3.2, C31.2, C33.2, C34.2, C35.2, C36.2, C4.2, C5.2, C6.2, C9.2, U2.22 (VS), U2.28 (VS), U3.22 (VS), U3.28 (VS), U4.3 (VI), U5.22 (VS), U5.28 (VS), U6.22 (VS), U6.28 (VS), U7.22 (VS), U7.28 (VS)
- net GND: now also C10.2, C11.2, C13.2, C14.2, C18.2, C19.2, C20.1, C23.2, C24.2, C28.2, C29.2, C4.2, C5.2, C6.2, C9.2, R13.1, R14.2, R18.2, R19.1, R21.1, R22.2, R23.1, R7.1, U5.9 (MS1_AD0), BT1.2 (-), C17.2, C22.2, C27.2, C30.1, C32.2, U8.1 (GND); no longer C13.1, C16.1, C18.1, C19.1, C24.1, C28.1, C3.1, C31.1, C33.1, C34.1, C36.1, C37.1, C4.1, C5.1, C6.1, R12.1, R16.2, R20.1, R21.2, R22.1, U6.9 (MS1_AD0)
- net RXD0: now also R12.2, R16.2, R20.2, R6.2, U2.14 (PDN_UART), U3.14 (PDN_UART), U5.14 (PDN_UART), U6.14 (PDN_UART); no longer R14.2, R19.2, R24.2, R7.2
- net RXD1: now also R24.2, U7.14 (PDN_UART)
- net TXD0: now also R12.1, R16.1, R20.1; no longer R13.1, R18.1, R23.1
- net TXD1: now also R24.1
- net at U2.4 (CP0): now also C3.2; no longer C11.1
- net at U2.5 (CPI): now also C3.1; no longer C11.2
- net at U3.27 (BRB): now also R14.1; no longer R16.1
- net at U5.1 (OB2): now also J4.4 (Pin_4); no longer J5.4 (Pin_4)
- net at U5.2 (ENN): now also R15.2; no longer R17.2
- net at U5.21 (OA2): now also J4.2 (Pin_2); no longer J5.2 (Pin_2)
- net at U5.23 (BRA): now also R17.2; no longer R20.2
- net at U5.24 (OA1): now also J4.1 (Pin_1); no longer J5.1 (Pin_1)
- net at U5.26 (OB1): now also J4.3 (Pin_3); no longer J5.3 (Pin_3)
- net at U5.27 (BRB): now also R18.1; no longer R21.1
- net at U5.4 (CP0): now also C21.2; no longer C29.1
- net at U5.5 (CPI): now also C21.1; no longer C29.2
- net at U5.8 (5VOUT): now also C22.1
- net at U6.1 (OB2): now also J5.4 (Pin_4); no longer J6.4 (Pin_4)
- net at U6.2 (ENN): now also R19.2; no longer R22.2
- net at U6.21 (OA2): now also J5.2 (Pin_2); no longer J6.2 (Pin_2)
- net at U6.23 (BRA): now also R21.2; no longer R25.2
- net at U6.24 (OA1): now also J5.1 (Pin_1); no longer J6.1 (Pin_1)
- net at U6.26 (OB1): now also J5.3 (Pin_3); no longer J6.3 (Pin_3)
- net at R26.1: now also U7.27 (BRB); no longer U6.27 (BRB)
- net at U6.4 (CP0): now also C26.2
- net at U6.5 (CPI): now also C26.1
- net at C35.1: now also U5.6 (VCP); no longer U6.6 (VCP)
- net at U6.8 (5VOUT): now also C27.1
- net at U7.6 (VCP): now also C37.1
- net at U3.2 (ENN): now also R7.2; no longer R12.2
- net at U3.1 (OB2): now also J1.4 (Pin_4); no longer J4.4 (Pin_4)
- net at U3.21 (OA2): now also J1.2 (Pin_2); no longer J4.2 (Pin_2)
- net at U3.23 (BRA): now also R13.2; no longer R15.2
- net at U3.24 (OA1): now also J1.1 (Pin_1); no longer J4.1 (Pin_1)
- net at U3.26 (OB1): now also J1.3 (Pin_3); no longer J4.3 (Pin_3)
- net at U3.4 (CP0): now also C16.2; no longer C20.1
- net at U3.5 (CPI): now also C16.1; no longer C20.2
- net at U3.6 (VCP): now also C34.1; no longer C14.1
- net at U3.8 (5VOUT): now also C17.1
- net at U7.4 (CP0): now also C31.2
- net at U7.5 (CPI): now also C31.1
- net at U7.23 (BRA): now also R25.2
- net at U7.2 (ENN): now also R23.2
- net at U7.24 (OA1): now also J6.1 (Pin_1)
- net at U7.21 (OA2): now also J6.2 (Pin_2)
- net at U7.26 (OB1): now also J6.3 (Pin_3)
- net at U7.1 (OB2): now also J6.4 (Pin_4)
- net at U7.8 (5VOUT): now also C32.1
- net IO19 renamed D-
- net IO20 renamed D+
- net IO47 renamed PWM
- new net: C33.1, U2.6 (VCP)
- new net: C36.1, U6.6 (VCP)
- new net: C10.1, J2.A4 (VBUS), J2.A9 (VBUS), J2.B4 (VBUS), J2.B9 (VBUS), U8.3 (VI)
- new net: R22.1, U6.27 (BRB)
- new net VBAT: BT1.1 (+), C13.1, C14.1, C18.1, C19.1, C23.1, C24.1, C28.1, C29.1, C33.2, C34.2, C35.2, C36.2, C37.2, C4.1, C5.1, C6.1, U2.22 (VS), U2.28 (VS), U3.22 (VS), U3.28 (VS), U4.3 (VI), U5.22 (VS), U5.28 (VS), U6.22 (VS), U6.28 (VS), U7.22 (VS), U7.28 (VS)
Other:
- moved on the sheet: C1, C12, C2, C49, C50, C7, C8, J2, J3, J8, R1, R10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

Commit message: Add files via upload
Connections:
- net +5V is gone; now on net VBAT: C49.1, C50.1, J8.1 (Pin_1)
Other:
- note added: "BATTERY"
- note added: "SERVO"
- note added: "STEPPER J1"
- note added: "STEPPER J2"
- note added: "STEPPER J3"
- note added: "STEPPER J4"
- note added: "STEPPER J5"
- note added: "USBC"

Commit message: Add files via upload
Schematic
Parts:
- BT1: footprint (none) -> Connector_Phoenix_GMSTB:PhoenixContact_GMSTBVA_2,5_2-G-7,62_1x02_P7.62mm_Vertical
- C10, C11, C6, C9: footprint (none) -> Capacitor_SMD:C_0805_2012Metric
- C13, C18, C23, C28, C4: footprint (none) -> Capacitor_SMD:C_1206_3216Metric
- C14, C16, C19, C21, C24, C26, C29, C3, C31, C33, C34, C35, C36, C37, C5: footprint (none) -> Capacitor_SMD:C_0402_1005Metric
- J1, J3, J4, J5, J6: footprint (none) -> Connector_Phoenix_GMSTB:PhoenixContact_GMSTBVA_2,5_4-G-7,62_1x04_P7.62mm_Vertical
- J2: footprint (none) -> Connector_USB:USB_C_Receptacle_GCT_USB4105-xx-A_16P_TopMnt_Horizontal
- J8: footprint (none) -> Connector_Phoenix_GMSTB:PhoenixContact_GMSTBVA_2,5_3-G-7,62_1x03_P7.62mm_Vertical
- SW1, SW2: footprint (none) -> Button_Switch_SMD:SW_Push_1P1T_NO_CK_KMR2
- U1: footprint (none) -> RF_Module:ESP32-S3-WROOM-1
- U2, U3, U5, U6, U7: footprint (none) -> MyFootprintLibrary:tmc2209
Connections:
- net GND: now also U2.25 (GND), U2.29 (GND), U3.29 (GND), U5.29 (GND), U6.29 (GND), U7.29 (GND)
Other:
- moved on the sheet: R12, R16, R20, R24, R6

Commit message: Add files via upload
Parts:
- removed BT1: Battery, Connector_Phoenix_GMSTB:PhoenixContact_GMSTBVA_2,5_2-G-7,62_1x02_P7.62mm_Vertical, symbol Device:Battery
- removed C13, C18, C23, C28, C4, C49: 100μF, Capacitor_SMD:C_1206_3216Metric, symbol Device:C_Small
- removed C50: 100nF, Capacitor_SMD:C_0402_1005Metric, symbol Device:C_Small
- removed R12, R16, R20, R24, R6: 1K, Resistor_SMD:R_0402_1005Metric, symbol Device:R
- removed R15, R19, R23, R5, R7: 10K, Resistor_SMD:R_0402_1005Metric, symbol Device:R
- added C13, C18, C23, C38, C4: 100μF, Capacitor_Tantalum_SMD:CP_EIA-6032-28_Kemet-C, symbol Device:C_Polarized
- added C28: 100uF, Capacitor_Tantalum_SMD:CP_EIA-6032-28_Kemet-C, symbol Device:C_Polarized
- added C39: 100nF, Capacitor_SMD:C_0402_1005Metric, symbol Device:C
- added D1, D2: PMEG3010EJ, Diode_SMD:D_SOD-123, symbol Device:D
- added J7: Screw_Terminal_01x02, Connector_Phoenix_GMSTB:PhoenixContact_GMSTBVA_2,5_2-G-7,62_1x02_P7.62mm_Vertical, symbol Connector:Screw_Terminal_01x02
- added R27, R28: 100K, Resistor_SMD:R_0402_1005Metric, symbol Device:R
- added R29, R30: 1K, Resistor_SMD:R_0402_1005Metric, symbol Device:R
- added U10, U9: TVS1400DRV, Package_SON:WSON-6-1EP_2x2mm_P0.65mm_EP1x1.6mm, symbol Power_Protection:TVS1400DRV
Connections:
- net +3V3: now also D1.1 (K), D2.1 (K), R27.2, R28.2; no longer C11.1, C9.1, U4.2 (VO), U8.2 (VO)
- net GND: now also U3.25 (GND), U5.25 (GND), U6.25 (GND), U7.25 (GND), C13.2, C18.2, C23.2, C28.2, C38.2, C39.2, C4.2, J7.1 (Pin_1), U10.1 (GND), U10.2 (GND), U10.3 (GND), U10.7 (GND), U9.1 (GND), U9.2 (GND), U9.3 (GND), U9.7 (GND)
- net TXD0: now also R29.2
- net TXD1: now also R30.2
- net VBAT: now also C13.1, C18.1, C23.1, C28.1, C38.1, C39.1, C4.1, J7.2 (Pin_2), U9.4 (IN), U9.5 (IN), U9.6 (IN)
- net ENN: now reaches U2.2 (ENN)
- net ENN: now also U1.22 (IO14), U3.2 (ENN), U5.2 (ENN), U6.2 (ENN), U7.2 (ENN)
- net at C10.1, J2.A4 (VBUS), J2.A9 (VBUS)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: now also U10.4 (IN), U10.5 (IN), U10.6 (IN)
- net RXD0 renamed PDN0-TX
- net PDN0-TX: now also R27.1, R29.1
- net RXD1 renamed PDN1-TX
- net PDN1-TX: now also R28.1, R30.1
- new net: C9.1, D2.2 (A), U4.2 (VO)
- new net: C11.1, D1.2 (A), U8.2 (VO)
- no-connect marks 18 -> 17
Other:
- note added: "CONNECTOR"
- note added: "UART03V3-RX"
- note added: "UART03V3-TX"
- note added: "UART13V3-RX"
- note added: "UART13V3-TX"
- moved on the sheet: C10, C11, C6, C9, J8, U2, U3, U4, U5, U6, U7, U8

Commit message: Add files via upload
Other:
- note added: "ESP32"
Changed lines of the file:
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@@
+		)
+	)
+	(text "ESP32\n"
+		(exclude_from_sim no)
+		(at 17.272 169.672 0)
+		(effects
+			(font
+				(size 1.27 1.27)
+			)
 		)
 	)
