File: Stasis-Robotic-Arm/Stasis-Robotic-Arm-CURRENT.kicad_sch (KiCad schematic)
At the start: 81 parts, among them J1 Screw_Terminal_01x04, J2 USB_C_Receptacle_USB2.0_14P, J3 Screw_Terminal_01x04, J4 Screw_Terminal_01x04, J5 Screw_Terminal_01x04, J6 Screw_Terminal_01x04, J7 Screw_Terminal_01x02, J8 Screw_Terminal_01x03, SW1 Enable, SW2 boot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

Commit message: Add files via upload
Parts:
- removed R8, R9: 22, Resistor_SMD:R_0402_1005Metric, symbol Device:R
- U1, U2, U3, U5, U6, U7: value ~ -> (none)
Connections:
- net +3V3: no longer C25.2, U6.15 (VCC_IO)
- net D+: now also J2.A6 (D+), J2.B6 (D+)
- net D-: now also J2.A7 (D-), J2.B7 (D-)
- new net: C25.2, U6.15 (VCC_IO)

Commit message: Add files via upload
Connections:
- net at U2.1 (OB2): now also J3.1 (Pin_1); no longer J3.4 (Pin_4)
- net at U2.21 (OA2): now also J3.4 (Pin_4); no longer J3.2 (Pin_2)
- net at U2.24 (OA1): now also J3.3 (Pin_3); no longer J3.1 (Pin_1)
- net at U2.26 (OB1): now also J3.2 (Pin_2); no longer J3.3 (Pin_3)
- net at U5.1 (OB2): now also J4.1 (Pin_1); no longer J4.4 (Pin_4)
- net at U5.21 (OA2): now also J4.4 (Pin_4); no longer J4.2 (Pin_2)
- net at U5.24 (OA1): now also J4.3 (Pin_3); no longer J4.1 (Pin_1)
- net at U5.26 (OB1): now also J4.2 (Pin_2); no longer J4.3 (Pin_3)
- net at J5.1 (Pin_1): now also U6.1 (OB2); no longer U6.24 (OA1)
- net at J5.2 (Pin_2): now also U6.26 (OB1); no longer U6.21 (OA2)
- net at J5.3 (Pin_3): now also U6.24 (OA1); no longer U6.26 (OB1)
- net at J5.4 (Pin_4): now also U6.21 (OA2); no longer U6.1 (OB2)
- net at U7.1 (OB2): now also J6.1 (Pin_1); no longer J6.4 (Pin_4)
- net at U7.21 (OA2): now also J6.4 (Pin_4); no longer J6.2 (Pin_2)
- net at U7.24 (OA1): now also J6.3 (Pin_3); no longer J6.1 (Pin_1)
- net at U7.26 (OB1): now also J6.2 (Pin_2); no longer J6.3 (Pin_3)
- net at U3.1 (OB2): now also J1.1 (Pin_1); no longer J1.4 (Pin_4)
- net at U3.21 (OA2): now also J1.4 (Pin_4); no longer J1.2 (Pin_2)
- net at U3.24 (OA1): now also J1.3 (Pin_3); no longer J1.1 (Pin_1)
- net at U3.26 (OB1): now also J1.2 (Pin_2); no longer J1.3 (Pin_3)
Changed lines of the file:
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@@
 	)
 	(symbol
-		(lib_name "TMC2209_1")
 		(lib_id "My-Kicad-Library:TMC2209")
 		(at 234.95 67.31 0)
@@
 	)
 	(symbol
-		(lib_name "TMC2209_3")
 		(lib_id "My-Kicad-Library:TMC2209")
 		(at 234.95 135.89 0)
@@
 	)
 	(symbol
-		(lib_name "TMC2209_4")
 		(lib_id "My-Kicad-Library:TMC2209")
 		(at 234.95 204.47 0)
@@
 	)
 	(symbol
-		(lib_name "TMC2209_2")
 		(lib_id "My-Kicad-Library:TMC2209")
 		(at 350.52 67.31 0)

Commit message: Add files via upload
Connections:
- net +3V3: now also C25.2, U6.15 (VCC_IO)
- net DIAG_1: now also U1.30 (IO37); no longer U1.23 (IO21)
- net DIAG_4: now also U1.33 (IO40); no longer U1.38 (IO2)
- net DIAG_5: now also U1.34 (IO41); no longer U1.39 (IO1)
- net DIR_1: now also U1.15 (IO3); no longer U1.5 (IO5)
- net DIR_2: now also U1.17 (IO9); no longer U1.7 (IO7)
- net DIR_3: now also U1.19 (IO11); no longer U1.16 (IO46)
- net DIR_4: now also U1.21 (IO13); no longer U1.18 (IO10)
- net DIR_5: now also U1.23 (IO21); no longer U1.20 (IO12)
- net ENN: no longer U1.22 (IO14)
- net PDN-UART1: now also U1.38 (IO2); no longer U1.35 (IO42)
- net PWM: now also U1.25 (IO48); no longer U1.24 (IO47)
- net STEP_1: now also U1.16 (IO46); no longer U1.4 (IO4)
- net STEP_2: now also U1.18 (IO10); no longer U1.6 (IO6)
- net STEP_3: now also U1.20 (IO12); no longer U1.17 (IO9)
- net STEP_4: now also U1.22 (IO14); no longer U1.19 (IO11)
- net STEP_5: now also U1.24 (IO47); no longer U1.21 (IO13)
- net TXD1: now also U1.35 (IO42); no longer U1.34 (IO41)
- no-connect marks 17 -> 18

Commit message: Add files via upload
Connections:
- net DIAG_1: now also U1.34 (IO41); no longer U1.30 (IO37)
- net DIAG_2: now also U1.33 (IO40); no longer U1.31 (IO38)
- net DIAG_4: now also U1.31 (IO38); no longer U1.33 (IO40)
- net DIAG_5: now also U1.30 (IO37); no longer U1.34 (IO41)
- net PDN-UART0: now also U1.38 (IO2); no longer U1.36 (RXD0)
- net PDN-UART1: now also U1.36 (RXD0); no longer U1.38 (IO2)
Changed lines of the file:
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@@
 	)
 	(label "DIAG_2"
-		(at 77.47 123.19 180)
+		(at 77.47 128.27 180)
 		(effects
 			(font
@@
 	)
 	(label "RXD0"
-		(at 77.47 140.97 180)
+		(at 77.47 135.89 180)
 		(effects
 			(font
@@
 	)
 	(label "DIAG_1"
-		(at 77.47 120.65 180)
+		(at 77.47 130.81 180)
 		(effects
 			(font
@@
 	)
 	(label "DIAG_4"
-		(at 77.47 128.27 180)
+		(at 77.47 123.19 180)
 		(effects
 			(font
@@
 	)
 	(label "DIAG_5"
-		(at 77.47 130.81 180)
+		(at 77.47 120.65 180)
 		(effects
 			(font
@@
 	)
 	(label "RXD1"
-		(at 77.47 135.89 180)
-		(effects
-			(font
+		(at 77.47 140.97 180)
+		(effects
+			(font
