File: Stasis-Robotic-Arm/StasisV3.kicad_pcb (KiCad board)
At the start: 2 copper layers, 78.2 x 56.9 mm, 75 parts, among them J1 MA, J2 MB, J3 MC, J4 MD, J5 ME, J6 SERVO, J7 POWER, J8 USB_C_Receptacle_USB2.0_14P, SW1 RST, SW2 BOOT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

Commit message: Add files via upload
Parts:
- added REF**: MountingHole_3.2mm_M3, MountingHole:MountingHole_3.2mm_M3, F.Cu at (124.3, 139.9)
- added REF**: MountingHole_3.2mm_M3, MountingHole:MountingHole_3.2mm_M3, F.Cu at (124.4, 89.3)
- added REF**: MountingHole_3.2mm_M3, MountingHole:MountingHole_3.2mm_M3, F.Cu at (196.2, 139.9)
- added REF**: MountingHole_3.2mm_M3, MountingHole:MountingHole_3.2mm_M3, F.Cu at (196.2, 88.8)
- moved J1 0.37 mm to (148.0, 137.7)
- moved J3 0.37 mm to (178.2, 137.7)
- moved J2 0.37 mm to (163.1, 137.7)
- moved C9 0.17 mm to (149.6, 126.7)
Connections:
- SW1 pad 2: GND -> Net-(U2-EN)
- SW2 pad 2: GND -> Net-(U2-IO0)
Routing:
- net Net-(U8-VI): track 12.0 -> 22.9 mm
- net VBAT: track 195.5 -> 205.9 mm, vias 7 -> 9
- net /D+: track 12.9 -> 15.1 mm
- net Net-(U2-EN): track 21.6 -> 23.8 mm
Other:
- board size 78.2 x 56.9 mm -> 79 x 57.8 mm

Commit message: Add files via upload
Parts:
- moved REF** 2.40 mm to (194.4, 90.5)
- moved REF** 2.40 mm to (194.4, 138.2)
- moved C2 2.36 mm to (124.8, 125.5), turned to -90 degrees
- moved C10 2.14 mm to (126.1, 132.4)
- moved C11 2.14 mm to (126.1, 130.1)
- moved C3 2.14 mm to (126.3, 126.0)
- moved D1 2.14 mm to (125.4, 127.7)
- moved R1 2.14 mm to (126.2, 125.0)
- moved U10 2.14 mm to (129.9, 135.3)
- moved U8 2.14 mm to (132.2, 130.1)
- moved REF** 2.11 mm to (125.6, 138.2)
- moved REF** 1.73 mm to (125.6, 90.5)
- moved C1 1.73 mm to (123.3, 125.0), turned to 180 degrees
- moved C39 0.53 mm to (147.5, 99.1)
- moved C28 0.46 mm to (145.4, 96.6)
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Routing:
- net VBAT: track 205.9 -> 208.2 mm
- net Net-(U8-VI): track 22.9 -> 20.7 mm
- net +3V3: track 180.6 -> 178.7 mm
- net Net-(U2-EN): track 23.8 -> 22.2 mm
- net /OA2-B: track 10.0 -> 8.57 mm
- net /PWM: track 28.0 -> 26.7 mm

Commit message: Add files via upload
Routing:
- net GND: track 0.03 -> 0.00 mm, vias 1 -> 0
Other:
- board text added: "ACE6RINGS"

Commit message: Add files via upload
Parts:
- removed D1, D2: PMEG3010EJ, Diode_SMD:D_SOD-123
Connections:
- C11 pad 1: Net-(D1-A) -> +3V3
- C34 pad 1: Net-(D2-A) -> +3V3
- U7 pad 2: Net-(D2-A) -> +3V3
- U8 pad 2: Net-(D1-A) -> +3V3
Routing:
- net +3V3: track 178.7 -> 203.8 mm
- net Net-(D1-A): track 10.9 -> 0.00 mm
- net Net-(D2-A): track 10.5 -> 0.00 mm
